File: fujiBLEboard.brd (EAGLE design)
At the start: 30.5 x 17.8 mm, 17 parts, among them IC1 MCP1703CB, X1 ABS05-32.768KHZ-9-T

Commit message: some improvement
Changed lines of the file:
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@@
 <?xml version="1.0" encoding="utf-8"?>
 <!DOCTYPE eagle SYSTEM "eagle.dtd">
-<eagle version="8.4.3">
+<eagle version="9.0.0">
 <drawing>
 <settings>
@@
 <setting verticaltext="up"/>
 </settings>
-<grid distance="10" unitdist="mil" unit="mil" style="lines" multiple="1" display="yes" altdistance="5" altunitdist="mil" altunit="mil"/>
+<grid distance="0.1" unitdist="mm" unit="mm" style="lines" multiple="1" display="yes" altdistance="0.05" altunitdist="mm" altunit="mm"/>
 <layers>
 <layer number="1" name="Top" color="4" fill="1" visible="yes" active="yes"/>
@@
 <layer number="39" name="tKeepout" color="4" fill="11" visible="no" active="yes"/>
 <layer number="40" name="bKeepout" color="1" fill="11" visible="no" active="yes"/>
-<layer number="41" name="tRestrict" color="4" fill="10" visible="no" active="yes"/>
-<layer number="42" name="bRestrict" color="1" fill="10" visible="no" active="yes"/>
+<layer number="41" name="tRestrict" color="4" fill="10" visible="yes" active="yes"/>
+<layer number="42" name="bRestrict" color="1" fill="10" visible="yes" active="yes"/>
 <layer number="43" name="vRestrict" color="2" fill="10" visible="no" active="yes"/>
 <layer number="44" name="Drills" color="7" fill="1" visible="no" active="yes"/>
@@
 <dimension x1="0" y1="1.27" x2="30.48" y2="1.27" x3="15.24" y3="-2.032" textsize="0.8128" layer="47" visible="yes"/>
 <dimension x1="1.27" y1="0" x2="1.27" y2="17.78" x3="-2.286" y3="8.89" textsize="0.8128" layer="47" visible="yes"/>
+<rectangle x1="17.25" y1="7.4" x2="17.4" y2="8.3" layer="41"/>
+<rectangle x1="26.8" y1="14.5" x2="30.7" y2="14.6" layer="41"/>
+<rectangle x1="28.1" y1="-1.1" x2="28.2" y2="14.6" layer="41"/>
+<rectangle x1="22.7" y1="14.2" x2="22.8" y2="18.3" layer="42"/>
+<rectangle x1="22.7" y1="14.2" x2="22.8" y2="18.3" layer="41"/>
+<rectangle x1="28.1" y1="-1.1" x2="28.2" y2="19.4" layer="42"/>
+<rectangle x1="6.9" y1="2" x2="7.1" y2="3" layer="42"/>
 </plain>
 <attributes>
@@
 <param name="checkRestrict" value="0"/>
 <param name="checkStop" value="0"/>
+<param name="checkValues" value="0"/>
 <param name="useDiameter" value="13"/>
 <param name="maxErrors" value="50"/>
@@
 </element>
 <element name="U$2" library="logo" package="LOGO-20MM" value="" x="23.622" y="5.842"/>
-<element name="U$3" library="logo" package="LOGO-20MM" value="" x="2.286" y="8.382" rot="MR270"/>
+<element name="U$3" library="logo" package="LOGO-20MM" value="" x="2.286" y="8.382" rot="SMR270"/>
 </elements>
 <signals>
@@
 <via x="19.685" y="5.842" extent="1-16" drill="0.4" diameter="0.4"/>
 <via x="26.289" y="5.842" extent="1-16" drill="0.4" diameter="0.4"/>
-<via x="28.067" y="10.16" extent="1-16" drill="0.4" diameter="0.4"/>
+<via x="27.467" y="10.06" extent="1-16" drill="0.4" diameter="0.4"/>
 <via x="27.305" y="12.7" extent="1-16" drill="0.4" diameter="0.4"/>
 <via x="23.114" y="12.7" extent="1-16" drill="0.4" diameter="0.4"/>
@@
 <via x="10.541" y="5.08" extent="1-16" drill="0.4" diameter="0.4"/>
 <via x="9.652" y="5.08" extent="1-16" drill="0.4" diameter="0.4"/>
+<via x="21.982" y="16.732" extent="1-16" drill="0.4" diameter="0.4"/>
+<via x="15.248" y="2.21" extent="1-16" drill="0.4" diameter="0.4"/>
 </signal>
 <signal name="SWCLK">
